File: Hardware/KiCad-files/Door-Sensor-no-edge-rails.kicad_pcb (KiCad board)
At the start: 4 copper layers, 40.7 x 40.6 mm, 52 parts, among them J1 I2C-Conn, J2 PWR-SERIAL-CONN, J3 TC2030, J5 U.FL, Q1 AO3401A, SW1 SW_Reed, SW2 SW_SPST, U1 nRF52832-QFxx, Y1 32.768kHz, Y2 32MHz

Commit message: added software
Parts:
- removed mouse-bite-2mm-slot (x4): VAL**, Panelization:mouse-bite-2mm-slot
Other:
- board size 40.7 x 40.6 mm -> 28.4 x 28.4 mm
- board text removed: "Dr. Sens V1.0 – frz.icu/dr-sens"
- board text removed: "JLCJLCJLCJLC"
